File: Proprietary_RJ45/Proprietary_RJ45.kicad_pcb (KiCad board)
At the start: 2 copper layers, 62 x 34.5 mm, 7 parts, among them J1 SS-60000-009, J2 436500227, J3 SS-60000-009

Commit message: add 3D models to project
Changed lines of the file:
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@@
 			(outputformat 1)
 			(mirror no)
-			(drillshape 1)
+			(drillshape 0)
 			(scaleselection 1)
-			(outputdirectory "")
+			(outputdirectory "gerber/")
 		)
 	)
@@
 		(tags "436500227 ")
 		(property "Reference" "J2"
-			(at -1.339599 3.760201 180)
+			(at -1.5 0 180)
 			(unlocked yes)
 			(layer "F.SilkS")
@@
 		)
 		(embedded_fonts no)
+		(model "${KIPRJMOD} /../models/1x2_CONN.stp"
+			(offset
+				(xyz -1.5 -2 10)
+			)
+			(scale
+				(xyz 1 1 1)
+			)
+			(rotate
+				(xyz 90 -0 -0)
+			)
+		)
 	)
 	(footprint "MountingHole:MountingHole_2.7mm_M2.5"
@@
 			)
 		)
-		(property "Datasheet" "https://www.digikey.com/short/w0j1wq4d"
+		(property "Datasheet" "SS-60000-009"
 			(at 0 0 270)
 			(layer "F.Fab")
@@
 		)
 		(embedded_fonts no)
+		(model "${KIPRJMOD} /../models/SS-60000-009.step"
+			(offset
+				(xyz -3.5 -4.5 0)
+			)
+			(scale
+				(xyz 1 1 1)
+			)
+			(rotate
+				(xyz -90 -0 -0)
+			)
+		)
 	)
 	(footprint "footprints:CONN8_SS-60000_STW"
@@
 			)
 		)
-		(property "Datasheet" "https://www.digikey.com/short/w0j1wq4d"
+		(property "Datasheet" "SS-60000-009"
 			(at 0 0 90)
 			(layer "F.Fab")
@@
 		)
 		(embedded_fonts no)
+		(model "${KIPRJMOD} /../models/SS-60000-009.step"
+			(offset
+				(xyz -3.5 -4.5 0)
+			)
+			(scale
+				(xyz 1 1 1)
+			)
+			(rotate
+				(xyz -90 -0 -0)
+			)
+		)
 	)
 	(footprint "MountingHole:MountingHole_2.7mm_M2.5"
@@
 		)
 	)
+	(dimension
+		(type orthogonal)
+		(layer "F.SilkS")
+		(pts
+			(xy 96.5 71.5) (xy 158.5 71.5)
+		)
+		(height -4.5)
+		(orientation 0)
+		(format
+			(prefix "")
+			(suffix "")
+			(units 3)
+			(units_format 0)
+			(precision 4)
+			(suppress_zeroes yes)
+		)
+		(style
+			(thickness 0.1)
+			(arrow_length 1.27)
+			(text_position_mode 0)
+			(arrow_direction outward)
+			(extension_height 0.58642)
+			(extension_offset 0.5)
+			(keep_text_aligned yes)
+		)
+		(gr_text "62"
+			(at 127.5 65.9 0)
+			(layer "F.SilkS")
+			(effects
+				(font
+					(size 1 1)
+					(thickness 0.1)
+				)
+			)
+		)
+	)
+	(dimension
+		(type orthogonal)
+		(layer "F.SilkS")
+		(pts
+			(xy 96.5 71.5) (xy 96.5 106)
+		)
+		(height -5.5)
+		(orientation 1)
+		(format
+			(prefix "")
+			(suffix "")
+			(units 3)
+			(units_format 0)
+			(precision 4)
+			(suppress_zeroes yes)
+		)
+		(style
+			(thickness 0.1)
+			(arrow_length 1.27)
+			(text_position_mode 0)
+			(arrow_direction outward)
+			(extension_height 0.58642)
+			(extension_offset 0.5)
+			(keep_text_aligned yes)
+		)
+		(gr_text "34.5"
+			(at 89.9 88.75 90)
+			(layer "F.SilkS")
+			(effects
+				(font
+					(size 1 1)
+					(thickness 0.1)
+				)
+			)
+		)
+	)
