File: Proprietary_RJ45/Proprietary_RJ45.kicad_sch (KiCad schematic)
At the start: 7 parts, among them J1 SS-60000-009, J2 436500227, J3 SS-60000-009

Commit message: add 3D models to project
Parts:
- J1, J3: footprint CONN8_SS-60000_STW -> footprints:CONN8_SS-60000_STW
Changed lines of the file:
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@@
 			)
 		)
-		(property "Footprint" "CONN8_SS-60000_STW"
+		(property "Footprint" "footprints:CONN8_SS-60000_STW"
 			(at 140.97 53.34 0)
 			(effects
@@
 			)
 		)
-		(property "Datasheet" "https://www.digikey.com/short/w0j1wq4d"
+		(property "Datasheet" "SS-60000-009"
 			(at 140.97 53.34 0)
 			(effects
@@
 			)
 		)
-		(property "Footprint" "CONN8_SS-60000_STW"
+		(property "Footprint" "footprints:CONN8_SS-60000_STW"
 			(at 114.3 53.34 0)
 			(effects
@@
 			)
 		)
-		(property "Datasheet" "https://www.digikey.com/short/w0j1wq4d"
+		(property "Datasheet" "SS-60000-009"
 			(at 114.3 53.34 0)
 			(effects
